Commit message: second_commit

File: my_robot_description/urdf/camera.xacro (robot description, xacro)
@@ -10,5 +10,5 @@
             <box size="${camera_width} ${camera_length} ${camera_height}"/>
         </geometry>
-        <material name = "red"/>
+        <material name = "black"/>
         </visual>
         <collision>

Commit message: add lidar scripts

File: my_robot_description/urdf/camera.xacro (robot description, xacro)
@@ -10,5 +10,5 @@
             <box size="${camera_width} ${camera_length} ${camera_height}"/>
         </geometry>
-        <material name = "black"/>
+        <material name = "red"/>
         </visual>
         <collision>

File: my_robot_description/urdf/main.xacro (robot description, xacro)
@@ -4,4 +4,5 @@
     <xacro:include filename = "properties_gazebo.xacro" />
     <xacro:include filename = "camera.xacro" />
+    <xacro:include filename = "lidar.xacro" />
     <xacro:include filename = "my_robot.xacro" />
 </robot>

File: my_robot_description/urdf/properties.xacro (robot description, xacro)
@@ -6,4 +6,7 @@
     <material name = "black">
         <color rgba = "0 0 0 1"/>
+    </material>
+    <material name = "green">
+        <color rgba = "0 1 0 1"/>
     </material>
     <material name = "red">

File: my_robot_description/urdf/properties_gazebo.xacro (robot description, xacro)
@@ -3,10 +3,16 @@
   <gazebo reference="base_link">
     <material>Gazebo/Blue</material>
+    <mu1 value ="0.1"/>
+    <mu2 value = "0.1"/>
   </gazebo>
   <gazebo reference="right_wheel_link">
     <material>Gazebo/Black</material>
+    <mu1 value ="0.1"/>
+    <mu2 value = "0.1"/>
   </gazebo>
   <gazebo reference="left_wheel_link">
     <material>Gazebo/Black</material>
+    <mu1 value ="0.1"/>
+    <mu2 value = "0.1"/>
   </gazebo>
   <gazebo reference="caster_wheel_link">
@@ -17,4 +23,9 @@
   <gazebo reference="camera_link">
     <material>Gazebo/Red</material>
+    <mu1 value ="0.1"/>
+    <mu2 value = "0.1"/>
+  </gazebo>
+  <gazebo reference="lidar_link">
+    <material>Gazebo/Green</material>
     <mu1 value ="0.1"/>
     <mu2 value = "0.1"/>
